Commit message: Documentation complete
Doxygen style comments and README completed

File: urdf/cracker_box.urdf.xacro (robot description, xacro)
@@ -4,5 +4,5 @@
   <xacro:property name="width" value="0.06" />
   <xacro:property name="height" value="0.21" />
-  <xacro:property name="M" value="0.3" />
+  <xacro:property name="M" value="0.001" />
   <link name="cracker_box_base_link"/>
   <link name="cracker_box_link">
@@ -34,4 +34,10 @@
   <gazebo reference="cracker_box_link">
     <material>Gazebo/Red</material>
+    <kp>1000000.0</kp>
+    <kd>100.0</kd>
+    <mu1>100.0</mu1>
+    <mu2>100.0</mu2>
+    <maxVel>1.0</maxVel>
+    <minDepth>0.001</minDepth>
   </gazebo>
 </robot>
